File: Sim-module.kicad_pcb (KiCad board)
At the start: 2 copper layers, 42 x 34 mm, 31 parts, among them J1 1*02, J10 Conn_01x01, J11 Conn_01x01, J12 Conn_01x01, J2 Rand connector, J3 Conn_01x01, J4 Conn_01x01, J5 Conn_01x01, J6 Conn_01x01, J7 Conn_01x01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

Commit message: Add files via upload
Parts:
- added REF**: OSHW-Logo_7.5x8mm_SilkScreen, Symbol:OSHW-Logo_7.5x8mm_SilkScreen, B.Cu at (194.0, 57.5)
